Commit message: Updated udacity_bot

File: urdf/udacity_bot.xacro (robot description, xacro)
@@ -1,190 +1,256 @@
 <?xml version='1.0'?>
 <robot name="udacity_bot" xmlns:xacro="http://www.ros.org/wiki/xacro">
-  <xacro:include filename="$(find udacity_bot)/urdf/udacity_bot.gazebo" />
-  <link name="robot_footprint"></link>
-  <joint name="robot_footprint_joint" type="fixed">
+<xacro:include filename="$(find udacity_bot)/urdf/udacity_bot.gazebo" />
+  <link name="robot_footprint">
+    <origin xyz="0 0 0" rpy=" 0 0 0"/>
+  </link>
+  <link name='chassis'>
+    <pose>0 0 0 0 0 0</pose>
+    <inertial>
+      <mass value="15.0"/>
+      <origin xyz="0 0 -0.05" rpy="0 0 0"/>
+      <inertia ixx="0.365625" ixy="0" ixz="0" iyy="0.365625" iyz="0" izz="0.675" />
+    </inertial>
+    <collision name='chassis_collision'>
+      <origin xyz="0 0 .015" rpy=" 0 0 0"/>
+      <geometry>
+        <cylinder radius=".3" length=".15"/>
+      </geometry>
+    </collision>
+    <visual name='chassis_visual'>
+      <origin xyz="0 0 .015" rpy=" 0 0 0"/>
+      <geometry>
+        <cylinder radius=".3" length=".15"/>
+      </geometry>
+      <material name="black_metal">
+	<color rgba="0.1 0.1 0.1 1"/>
+      </material>
+    </visual>
+    <visual name='chassis_dome_visual'>
+      <origin xyz="-0.2 0 0.11" rpy=" 0 0 0"/>
+      <geometry>
+        <cylinder radius=".05" length=".05"/>
+      </geometry>
+      <material name="black_metal">
+	<color rgba="0.1 0.1 0.1 1"/>
+      </material>
+    </visual>
+  </link>
+  <joint name="chassis_joint" type="fixed">
     <origin xyz="0 0 0" rpy="0 0 0" />
     <parent link="robot_footprint"/>
     <child link="chassis" />
   </joint>
-  <link name='chassis'>
-    <pose>0 0 0.1 0 0 0</pose>
-    <inertial>
-      <mass value="15.0"/>
+  <link name="camera_link">
+    <origin xyz="0 0 0" rpy="0 0 0"/>
+    <inertial>
+      <mass value="0.1"/>
+      <origin xyz="0 0 0" rpy="0 0 0"/>
+      <inertia ixx="1e-6" ixy="0" ixz="0" iyy="1e-6" iyz="0" izz="1e-6" />
+    </inertial>
+    <collision name='camera_collision'>
+      <origin xyz="0 0 0" rpy=" 0 0 0"/>
+      <geometry>
+        <box size="0.05 0.05 0.05"/>
+      </geometry>
+    </collision>
+    <visual name='camera_visual'>
+      <origin xyz="0 0 0" rpy=" 0 0 0"/>
+      <geometry>
+        <box size="0.05 0.05 0.05"/>
+      </geometry>
+    </visual>
+  </link>
+   <joint name="camera_joint" type="fixed">
+      <origin xyz="0.3 0 0" rpy="0 0 0"/>
+      <child link="camera_link"/>
+      <parent link="chassis"/>
+      <axis xyz="0 1 0" rpy="0 0 0"/>
+    <!--
+    <limit effort="10000" velocity="1000"/>
+    <dynamics damping="1.0" friction="1.0"/>
+    -->
+   </joint>
+  <link name="camera_link_optical"></link>
+   <joint name="camera_optical_joint" type="fixed" >
+      <origin xyz="0.3 0 0" rpy="-1.5707 0 -1.5707"/>
+      <parent link="camera_link"/>
+      <child link="camera_link_optical"/>
+   </joint>
+  <link name='front_caster'>
+    <pose>0 0 0 0 0 0</pose>
+    <inertial>
+      <origin xyz="0 0 0" rpy=" 0 0 0"/>
+      <mass value="2.0"/>
+      <inertia ixx="0.002" ixy="0" ixz="0" iyy="0.002" iyz="0" izz="0.002" />
+    </inertial>
+    <collision name='front_caster_collision'>
+      <origin xyz="0 0 0" rpy=" 0 0 0"/>
+      <geometry>
+        <sphere radius="0.05"/>
+      </geometry>
+      <surface>
+        <friction>
+          <ode>
+            <mu>0</mu>
+            <mu2>0</mu2>
+            <slip1>1.0</slip1>
+            <slip2>1.0</slip2>
+          </ode>
+        </friction>
+      </surface>
+    </collision>
+    <visual name='front_caster_visual'>
+      <origin xyz="0 0 0" rpy=" 0 0 0"/>
+      <geometry>
+        <sphere radius="0.05"/>
+      </geometry>
+      <material name="black_metal">
+	<color rgba="0.1 0.1 0.1 1"/>
+      </material>
+    </visual>
+  </link>
+   <joint type="continuous" name="front_caster_hinge">
+       <origin xyz="0.2 0 -0.05" rpy="0 0 0"/>
+       <parent link="chassis"/>
+       <child link="front_caster"/>
+       <axis xyz="0 1 0" rpy="0 0 0"/>
+       <limit effort="10000" velocity="1000"/>
+       <joint_properties damping="1.0" friction="1.0"/>
+   </joint>
+  <link name='back_caster'>
+    <pose>0 0 0 0 0 0</pose>
+    <inertial>
+      <origin xyz="0 0 0" rpy=" 0 0 0"/>
+      <mass value="2.0"/>
+      <inertia
+          ixx="0.002" ixy="0" ixz="0"
+          iyy="0.002" iyz="0"
+          izz="0.002"
+      />
+    </inertial>
+    <collision name='back_caster_collision'>
+      <origin xyz="0 0 0" rpy=" 0 0 0"/>
+      <geometry>
+        <sphere radius="0.05"/>
+      </geometry>
+      <surface>
+        <friction>
+          <ode>
+            <mu>0</mu>
+            <mu2>0</mu2>
+            <slip1>1.0</slip1>
+            <slip2>1.0</slip2>
+          </ode>
+        </friction>
+      </surface>
+    </collision>
+    <visual name='back_caster_visual'>
+      <origin xyz="0 0 0" rpy=" 0 0 0"/>
+      <geometry>
+        <sphere radius="0.05"/>
+      </geometry>
+      <material name="black_metal">
+	<color rgba="0.1 0.1 0.1 1"/>
+      </material>
+    </visual>
+  </link>
+   <joint type="continuous" name="back_caster_hinge">
+       <origin xyz="-0.2 0 -0.05" rpy="0 0 0"/>
+       <parent link="chassis"/>
+       <child link="back_caster"/>
+       <axis xyz="0 1 0" rpy="0 0 0"/>
+       <limit effort="10000" velocity="1000"/>
+       <joint_properties damping="1.0" friction="1.0"/>
+   </joint>
+  <link name='left_wheel'>
+    <pose>0 0 0 0 0 0</pose>
+    <inertial>
+      <origin xyz="0 0 0" rpy="0 1.57 1.57"/>
+      <mass value="2.0"/>
+      <inertia ixx="0.00185" ixy="0" ixz="0" iyy="0.00185" iyz="0" izz="0.0025" />
+    </inertial>
+    <collision name='left_wheel_collision'>
+      <origin xyz="0 0 0" rpy="0 1.57 1.57"/>
+      <geometry>
+        <cylinder radius=".05" length=".06"/>
+      </geometry>
+    </collision>
+    <visual name='left_wheel_visual'>
+      <origin xyz="0 0 0" rpy="0 1.57 1.57"/>
+      <geometry>
+        <cylinder radius=".05" length=".06"/>
+      </geometry>
+    </visual>
+      <material name="gold">
+        <color rgba="1 0.549 0 1"/>
+      </material>
+  </link>
+   <joint type="continuous" name="left_wheel_hinge">
+       <origin xyz="0 0.2 -0.05" rpy="0 0 0"/>
+       <parent link="chassis"/>
+       <child link="left_wheel"/>
+       <axis xyz="0 1 0" rpy="0 0 0"/>
+       <limit effort="10000" velocity="1000"/>
+       <joint_properties damping="1.0" friction="1.0"/>
+   </joint>
+  <link name='right_wheel'>
+    <pose>0 0 0 0 0 0</pose>
+    <inertial>
+      <origin xyz="0 0 0" rpy="0 1.57 1.57"/>
+      <mass value="2.0"/>
+      <inertia ixx="0.00185" ixy="0" ixz="0" iyy="0.00185" iyz="0" izz="0.0025" />
+    </inertial>
+    <collision name='right_wheel_collision'>
+      <origin xyz="0 0 0" rpy="0 1.57 1.57"/>
+      <geometry>
+        <cylinder radius=".05" length=".06"/>
+      </geometry>
+    </collision>
+    <visual name='right_wheel_visual'>
+      <origin xyz="0 0 0" rpy="0 1.57 1.57"/>
+      <geometry>
+        <cylinder radius=".05" length=".06"/>
+      </geometry>
+      <material name="gold">
+        <color rgba="1 0.549 0 1"/>
+      </material>
+    </visual>
+  </link>
+   <joint type="continuous" name="right_wheel_hinge">
+       <origin xyz="0 -0.2 -0.05" rpy="0 0 0"/>
+       <parent link="chassis"/>
+       <child link="right_wheel"/>
+       <axis xyz="0 1 0" rpy="0 0 0"/>
+       <limit effort="10000" velocity="1000"/>
+       <joint_properties damping="1.0" friction="1.0"/>
+   </joint>
+  <link name="hokuyo">
+    <inertial>
+      <mass value="0.1"/>
       <origin xyz="0.0 0 0" rpy=" 0 0 0"/>
       <inertia
-          ixx="0.1" ixy="0" ixz="0"
-          iyy="0.1" iyz="0"
-          izz="0.1"
-      />
-    </inertial>
-    <collision name='collision'>
-      <origin xyz="0 0 0" rpy=" 0 0 0"/>
-      <geometry>
-        <box size=".4 .2 .1"/>
-      </geometry>
-    </collision>
-    <visual name='chassis_visual'>
-      <origin xyz="0 0 0" rpy="0 0 0"/>
-      <geometry>
-        <box size=".4 .2 .1"/>
-      </geometry>
-    </visual>
-    <collision name='back_caster_collision'>
-      <origin xyz="-0.15 0 -0.05" rpy="0 0 0"/>
-      <geometry>
-        <sphere radius="0.0499"/>
-      </geometry>
-    </collision>
-    <visual name='back_caster_visual'>
-      <origin xyz="-0.15 0 -0.05" rpy="0 0 0"/>
-      <geometry>
-        <sphere radius="0.05"/>
-      </geometry>
-    </visual>
-    <collision name='front_caster_collision'>
-      <origin xyz="0.15 0 -0.05" rpy="0 0 0"/>
-      <geometry>
-        <sphere radius="0.0499"/>
-      </geometry>
-    </collision>
-    <visual name='front_caster_visual'>
-      <origin xyz="0.15 0 -0.05" rpy="0 0 0"/>
-      <geometry>
-        <sphere radius="0.05"/>
-      </geometry>
-    </visual>
-  </link>
-  <link name="left_wheel">
-    <inertial>
-      <mass value="5.0"/>
-      <origin xyz="0.0 0 0" rpy="0 1.5707 1.5707"/>
-      <inertia
-          ixx="0.1" ixy="0" ixz="0"
-          iyy="0.1" iyz="0"
-          izz="0.1"
-      />
-    </inertial>
-    <collision>
-      <origin xyz="0 0 0" rpy="0 1.5707 1.5707"/>
-       <cylinder radius="0.1" length="0.05"/>
-      <geometry>
-       <cylinder radius="0.1" length="0.05"/>
-      </geometry>
-    </collision>
-    <visual>
-      <origin xyz="0 0 0" rpy="0 1.5707 1.5707"/>
-      <geometry>
-       <cylinder radius="0.1" length="0.05"/>
-      </geometry>
-      <material name="red"/>
-    </visual>
-    <joint type="continuous" name="left_wheel_hinge">
-      <origin xyz="0 0.15 0" rpy="0 0 0"/>
-      <child link="left_wheel"/>
+          ixx="1e-6" ixy="0" ixz="0" iyy="1e-6" iyz="0" izz="1e-6" />
+    </inertial>
+    <collision name='hokuyo_collision'>
+      <origin xyz="0 0 0" rpy=" 0 0 0"/>
+      <geometry>
+        <box size=".1 .1 .1"/>
+      </geometry>
+    </collision>
+    <visual name='hokuyo_visual'>
+      <origin xyz="0 0 0" rpy=" 0 0 0"/>
+      <geometry>
+        <mesh filename="package://udacity_bot/meshes/hokuyo.dae"/>
+      </geometry>
+    </visual>
+      <material name="black_metal">
+	<color rgba="0.1 0.1 0.1 1"/>
+      </material>
+  </link>
+   <joint type="fixed" name="hokuyo_joint">
+      <origin xyz="-0.2 0 0.16" rpy=" 0 0 0"/>
       <parent link="chassis"/>
-      <axis xyz="0 1 0" rpy="0 0 0"/>
-      <limit effort="10000" velocity="1000"/>
-      <joint_properties damping="1.0" friction="1.0"/>
-    </joint>
-  </link>
-  <link name="right_wheel">
-    <inertial>
-      <mass value="5.0"/>
-      <origin xyz="0.0 0 0" rpy="0 1.5707 1.5707"/>
-      <inertia
-          ixx="0.1" ixy="0" ixz="0"
-          iyy="0.1" iyz="0"
-          izz="0.1"
-      />
-    </inertial>
-    <collision>
-      <origin xyz="0 0 0" rpy="0 1.5707 1.5707"/>
-       <cylinder radius="0.1" length="0.05"/>
-      <geometry>
-       <cylinder radius="0.1" length="0.05"/>
-      </geometry>
-    </collision>
-    <visual>
-      <origin xyz="0 0 0" rpy="0 1.5707 1.5707"/>
-      <geometry>
-       <cylinder radius="0.1" length="0.05"/>
-      </geometry>
-      <material name="red"/>
-    </visual>
-  </link>
-  <joint type="continuous" name="left_wheel_hinge">
-    <origin xyz="0 0.15 0" rpy="0 0 0"/>
-    <child link="left_wheel"/>
-    <parent link="chassis"/>
-    <axis xyz="0 1 0" rpy="0 0 0"/>
-    <limit effort="10000" velocity="1000"/>
-    <joint_properties damping="1.0" friction="1.0"/>
-  </joint>
-  <joint type="continuous" name="right_wheel_hinge">
-    <origin xyz="0 -0.15 0" rpy="0 0 0"/>
-    <child link="right_wheel"/>
-    <parent link="chassis"/>
-    <axis xyz="0 1 0" rpy="0 0 0"/>
-    <limit effort="10000" velocity="1000"/>
-    <joint_properties damping="1.0" friction="1.0"/>
-  </joint>
-    <link name="camera">
-    <collision>
-      <origin xyz="0 0 0" rpy="0 0 0"/>
-      <geometry>
-        <box size="0.05 0.05 0.05"/>
-      </geometry>
-    </collision>
-    <visual>
-      <origin xyz="0 0 0" rpy="0 0 0"/>
-      <geometry>
-        <box size="0.05 0.05 0.05"/>
-      </geometry>
-      <material name="red"/>
-    </visual>
-    <inertial>
-      <mass value="0.1" />
-      <origin xyz="0 0 0" rpy="0 0 0"/>
-     <box_inertia m="0.1" x="0.05" y="0.05" z="0.05" />
-      <inertia ixx="1e-6" ixy="0" ixz="0" iyy="1e-6" iyz="0" izz="1e-6" />
-    </inertial>
-  </link>
-  <joint name="camera_joint" type="fixed">
-    <axis xyz="0 1 0" />
-    <origin xyz="0.2 0 0" rpy="0 0 0"/>
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